File: kicad/mainboard_v1_0/mainboard_v1_0.sch (KiCad schematic (older format))
At the start: 32 parts, among them J1 Conn_01x02, J2 Conn_01x06, J3 Conn_01x04, J4 Conn_01x04, J5 Conn_01x05, SW1 SW_DIP_x06, U1 stm32f4_disco_board, U2 74HC245, U3 LM2596_MODULE, U4 AMS1117-3.3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

Commit message: add diode & led status
Parts:
- removed C11: 100nF, Capacitor_THT:C_Radial_D8.0mm_H11.5mm_P3.50mm, symbol Device:C_Small
- removed U6: MPU_9250, Connector_PinHeader_2.54mm:PinHeader_1x10_P2.54mm_Vertical, symbol mpu_9250:MPU_9250
- added C2: 10uF, Capacitor_THT:C_Radial_D8.0mm_H11.5mm_P3.50mm, symbol Device:CP_Small
- added D1: SS24, Diode_SMD:D_SMA, symbol Device:D_Small
- added D2: LED_Small, LED_THT:LED_D3.0mm, symbol Device:LED_Small
- added J6: Conn_01x08, Connector_PinHeader_2.54mm:PinHeader_1x08_P2.54mm_Vertical, symbol Connector_Generic:Conn_01x08
- added JP2: Jumper, Connector_PinHeader_2.54mm:PinHeader_1x02_P2.54mm_Vertical, symbol Device:Jumper
- added R2: R_Small, Resistor_THT:R_Axial_DIN0207_L6.3mm_D2.5mm_P10.16mm_Horizontal, symbol Device:R_Small
Connections:
- net labels added: MPU_6050_SCL, MPU_6050_SDA, VMCU
- net labels removed: MPU_9250_SCL, MPU_9250_SDA
- wire segments 133 -> 131
Other:
- moved on the sheet: C14, U3
Changed lines of the file:
@@
-$EndComp
-$Comp
-L mpu_9250:MPU_9250 U6
-U 1 1 5DFE3356
-P 6400 7500
-F 0 "U6" H 6600 8650 50  0000 L CNN
-F 1 "MPU_9250" H 6150 8650 50  0000 L CNN
-F 2 "Connector_PinHeader_2.54mm:PinHeader_1x10_P2.54mm_Vertical" H 6250 7900 50  0001 C CNN
-F 3 "" H 6250 7900 50  0001 C CNN
-	1    6400 7500
-	1    0    0    -1
 $EndComp
 $Comp
@@
 	1    0    0    -1
 $EndComp
-$Comp
-L Device:C_Small C11
-U 1 1 5E08D010
-P 7800 1500
-F 0 "C11" H 7892 1546 50  0000 L CNN
-F 1 "100nF" H 7892 1455 50  0000 L CNN
-F 2 "Capacitor_THT:C_Radial_D8.0mm_H11.5mm_P3.50mm" H 7800 1500 50  0001 C CNN
-F 3 "~" H 7800 1500 50  0001 C CNN
-	1    7800 1500
-	1    0    0    -1
-$EndComp
-Wire Wire Line
-	7800 1350 7800 1400
-Wire Wire Line
-	7800 1650 7800 1600
 Wire Wire Line
 	7450 2300 7450 2350
@@
 $EndComp
 $Comp
-L power:GND #PWR021
-U 1 1 5E098307
-P 7650 1650
-F 0 "#PWR021" H 7650 1400 50  0001 C CNN
-F 1 "GND" H 7655 1477 50  0000 C CNN
-F 2 "" H 7650 1650 50  0001 C CNN
-F 3 "" H 7650 1650 50  0001 C CNN
-	1    7650 1650
-	1    0    0    -1
-$EndComp
-Wire Wire Line
-	7650 1650 7800 1650
-$Comp
 L power:+5V #PWR017
 U 1 1 5E0987CC
@@
 	1    0    0    -1
 $EndComp
-Text GLabel 7650 1300 1    50   Input ~ 0
-VMOT
-Wire Wire Line
-	7650 1300 7650 1350
-Wire Wire Line
-	7650 1350 7800 1350
 Text GLabel 9350 1000 0    50   Input ~ 0
 VMOT
@@
 L Device:CP_Small C14
 U 1 1 5E0E8BC5
-P 9850 1600
-F 0 "C14" H 9938 1646 50  0000 L CNN
-F 1 "10uF" H 9938 1555 50  0000 L CNN
-F 2 "Capacitor_THT:C_Radial_D8.0mm_H11.5mm_P3.50mm" H 9850 1600 50  0001 C CNN
-F 3 "~" H 9850 1600 50  0001 C CNN
-	1    9850 1600
-	1    0    0    -1
-$EndComp
-Wire Wire Line
-	9850 1500 9850 1450
-Wire Wire Line
-	9850 1450 10000 1450
-Wire Wire Line
-	9850 1700 9850 1750
-Wire Wire Line
-	9850 1750 10000 1750
+P 10000 1610
+F 0 "C14" H 10088 1656 50  0000 L CNN
+F 1 "10uF" H 10088 1565 50  0000 L CNN
+F 2 "Capacitor_THT:C_Radial_D8.0mm_H11.5mm_P3.50mm" H 10000 1610 50  0001 C CNN
+F 3 "~" H 10000 1610 50  0001 C CNN
+	1    10000 1610
+	1    0    0    -1
+$EndComp
 Wire Wire Line
 	9800 2400 9800 2450
@@
 Text GLabel 10000 1400 1    50   Input ~ 0
 VMOT
-Wire Wire Line
-	10000 1400 10000 1450
 Wire Wire Line
 	9800 4000 9800 4050
@@
 $EndComp
 Text GLabel 6200 6700 0    50   Input ~ 0
-MPU_9250_SCL
+MPU_6050_SCL
 Text GLabel 6200 6800 0    50   Input ~ 0
-MPU_9250_SDA
-Wire Wire Line
-	6200 6700 6300 6700
-Wire Wire Line
-	6200 6800 6300 6800
+MPU_6050_SDA
 $Comp
 L power:+3V3 #PWR012
@@
 UART_ROS_TX
 Text GLabel 4650 2200 2    50   Input ~ 0
-MPU_9250_SDA
+MPU_6050_SDA
 Text GLabel 3900 2200 0    50   Input ~ 0
-MPU_9250_SCL
+MPU_6050_SCL
 Text GLabel 1950 1700 0    50   Input ~ 0
 MOTOR_2_DIR
@@
 MOTOR_1_PULSE
 $Comp
-L power:+5V #PWR0101
-U 1 1 5E5B85DF
-P 3900 1200
-F 0 "#PWR0101" H 3900 1050 50  0001 C CNN
-F 1 "+5V" H 3915 1373 50  0000 C CNN
-F 2 "" H 3900 1200 50  0001 C CNN
-F 3 "" H 3900 1200 50  0001 C CNN
-	1    3900 1200
-	0    -1   -1   0
-$EndComp
-$Comp
 L power:GND #PWR0102
 U 1 1 5E5B8D51
 P 3900 1100
 F 0 "#PWR0102" H 3900 850 50  0001 C CNN
-F 1 "GND" H 3905 927 50  0000 C CNN
+F 1 "GND" V 3905 927 50  0000 C CNN
 F 2 "" H 3900 1100 50  0001 C CNN
 F 3 "" H 3900 1100 50  0001 C CNN
@@
 L lm2596_module:LM2596_MODULE U3
 U 1 1 5E12ED1D
-P 3945 6710
-F 0 "U3" H 4185 6906 50  0000 L CNN
-F 1 "LM2596_MODULE" H 4185 6815 50  0000 L CNN
-F 2 "footprints:LM2596_MODULE" H 3945 6710 50  0001 C CNN
-F 3 "" H 3945 6710 50  0001 C CNN
-	1    3945 6710
+P 3390 6515
+F 0 "U3" H 3630 6711 50  0000 L CNN
+F 1 "LM2596_MODULE" H 3630 6620 50  0000 L CNN
+F 2 "footprints:LM2596_MODULE" H 3390 6515 50  0001 C CNN
+F 3 "" H 3390 6515 50  0001 C CNN
+	1    3390 6515
 	1    0    0    -1
 $EndComp
@@
 	1    0    0    -1
 $EndComp
+$Comp
+L Device:D_Small D1
+U 1 1 5E1903CA
+P 5240 1615
+F 0 "D1" H 5340 1570 50  0000 C CNN
+F 1 "SS24" H 5255 1705 50  0000 C CNN
+F 2 "Diode_SMD:D_SMA" V 5240 1615 50  0001 C CNN
+F 3 "~" V 5240 1615 50  0001 C CNN
+	1    5240 1615
+	0    -1   -1   0
+$EndComp
+Wire Wire Line
+	3775 1200 3900 1200
+Wire Wire Line
+	10000 1400 10000 1510
+Wire Wire Line
+	10000 1710 10000 1750
+$Comp
+L Device:CP_Small C2
+U 1 1 5E1D2EB9
+P 7670 1550
+F 0 "C2" H 7758 1596 50  0000 L CNN
+F 1 "10uF" H 7758 1505 50  0000 L CNN
+F 2 "Capacitor_THT:C_Radial_D8.0mm_H11.5mm_P3.50mm" H 7670 1550 50  0001 C CNN
+F 3 "~" H 7670 1550 50  0001 C CNN
+	1    7670 1550
+	1    0    0    -1
+$EndComp
+$Comp
+L power:GND #PWR04
+U 1 1 5E1D2EBF
+P 7670 1690
+F 0 "#PWR04" H 7670 1440 50  0001 C CNN
+F 1 "GND" H 7675 1517 50  0000 C CNN
+F 2 "" H 7670 1690 50  0001 C CNN
+F 3 "" H 7670 1690 50  0001 C CNN
+	1    7670 1690
+	1    0    0    -1
+$EndComp
+Text GLabel 7670 1340 1    50   Input ~ 0
+VMOT
+Wire Wire Line
+	7670 1340 7670 1450
+Wire Wire Line
+	7670 1650 7670 1690
+$Comp
+L Device:LED_Small D2
+U 1 1 5E1EE5CB
+P 4520 7260
+F 0 "D2" V 4566 7192 50  0000 R CNN
+F 1 "LED_Small" V 4475 7192 50  0000 R CNN
+F 2 "LED_THT:LED_D3.0mm" V 4520 7260 50  0001 C CNN
+F 3 "~" V 4520 7260 50  0001 C CNN
+	1    4520 7260
+	0    -1   -1   0
+$EndComp
+$Comp
+L Device:R_Small R2
+U 1 1 5E1F7E2B
+P 4520 6965
+F 0 "R2" H 4579 7011 50  0000 L CNN
+F 1 "R_Small" H 4579 6920 50  0000 L CNN
+F 2 "Resistor_THT:R_Axial_DIN0207_L6.3mm_D2.5mm_P10.16mm_Horizontal" H 4520 6965 50  0001 C CNN
+F 3 "~" H 4520 6965 50  0001 C CNN
+	1    4520 6965
+	1    0    0    -1
+$EndComp
+Wire Wire Line
+	4520 7160 4520 7065
+$Comp
+L power:GND #PWR0106
+U 1 1 5E1FF088
+P 4520 7360
+F 0 "#PWR0106" H 4520 7110 50  0001 C CNN
+F 1 "GND" H 4525 7187 50  0000 C CNN
+F 2 "" H 4520 7360 50  0001 C CNN
+F 3 "" H 4520 7360 50  0001 C CNN
+	1    4520 7360
+	1    0    0    -1
+$EndComp
+$Comp
+L power:+3V3 #PWR0107
+U 1 1 5E2011D4
+P 4520 6865
+F 0 "#PWR0107" H 4520 6715 50  0001 C CNN
+F 1 "+3V3" H 4535 7038 50  0000 C CNN
+F 2 "" H 4520 6865 50  0001 C CNN
+F 3 "" H 4520 6865 50  0001 C CNN
+	1    4520 6865
+	1    0    0    -1
+$EndComp
+$Comp
+L Connector_Generic:Conn_01x08 J6
+U 1 1 5E20AA32
+P 6605 6800
+F 0 "J6" H 6685 6792 50  0000 L CNN
+F 1 "Conn_01x08" H 6685 6701 50  0000 L CNN
+F 2 "Connector_PinHeader_2.54mm:PinHeader_1x08_P2.54mm_Vertical" H 6605 6800 50  0001 C CNN
+F 3 "~" H 6605 6800 50  0001 C CNN
+	1    6605 6800
+	1    0    0    -1
+$EndComp
+Wire Wire Line
+	6300 6500 6405 6500
+Wire Wire Line
+	6300 6600 6405 6600
+Wire Wire Line
+	6200 6700 6405 6700
+Wire Wire Line
+	6200 6800 6405 6800
+$Comp
+L Device:Jumper JP2
+U 1 1 5E25D960
+P 5240 1215
+F 0 "JP2" H 5240 1479 50  0000 C CNN
+F 1 "Jumper" H 5240 1388 50  0000 C CNN
+F 2 "Connector_PinHeader_2.54mm:PinHeader_1x02_P2.54mm_Vertical" H 5240 1215 50  0001 C CNN
+F 3 "~" H 5240 1215 50  0001 C CNN
+	1    5240 1215
+	0    1    1    0
+$EndComp
+$Comp
+L power:+5V #PWR0101
+U 1 1 5E5B85DF
+P 5240 915
+F 0 "#PWR0101" H 5240 765 50  0001 C CNN
+F 1 "+5V" H 5255 1088 50  0000 C CNN
+F 2 "" H 5240 915 50  0001 C CNN
+F 3 "" H 5240 915 50  0001 C CNN
+	1    5240 915
+	1    0    0    -1
+$EndComp
+Text GLabel 5240 1715 3    50   Input ~ 0
+VMCU
+Text GLabel 3775 1200 0    50   Input ~ 0
+VMCU
 $EndSCHEMATC

Commit message: update schematic
Parts:
- D1: footprint Diode_SMD:D_SMA -> Diode_THT:D_5W_P12.70mm_Horizontal
Changed lines of the file:
@@
 F 0 "D1" H 5340 1570 50  0000 C CNN
 F 1 "SS24" H 5255 1705 50  0000 C CNN
-F 2 "Diode_SMD:D_SMA" V 5240 1615 50  0001 C CNN
+F 2 "Diode_THT:D_5W_P12.70mm_Horizontal" V 5240 1615 50  0001 C CNN
 F 3 "~" V 5240 1615 50  0001 C CNN
 	1    5240 1615
