Commit message: update urdf description

File: ros/src/robot/robot_description/urdf/robot_thesis.urdf.xacro (robot description, xacro)
@@ -119,11 +119,11 @@
   </joint>
   <link name="base_scan">
-    <visual>
+    <!-- <visual>
       <origin xyz="0 0 0.0" rpy="0 0 0"/>
       <geometry>
-        <mesh filename="package://turtlebot3_description/meshes/sensors/lds.stl" scale="0.001 0.001 0.001"/>
+        <mesh filename="package://robot_description/meshes/stl/robot_lidar.stl" scale="0.001 0.001 0.001"/>
       </geometry>
       <material name="dark"/>
-    </visual>
+    </visual> -->
     <collision>
       <origin xyz="0.015 0 -0.0065" rpy="0 0 0"/>

Commit message: fix collision in urdf description

File: ros/src/robot/robot_description/urdf/robot_thesis.urdf.xacro (robot description, xacro)
@@ -11,5 +11,5 @@
   <link name="base_link">
     <visual>
-      <origin xyz="0 0 0.0525" rpy="0 0 -1.5707"/>
+      <origin xyz="-0.032 0 0.0525" rpy="0 0 -1.5707"/>
       <geometry>
         <mesh filename="package://robot_description/meshes/stl/robot_base.stl" scale="0.001 0.001 0.001"/>
@@ -18,7 +18,7 @@
     </visual>
     <collision>
-      <origin xyz="0      0      0.0925" rpy="0 0 0"/>
+      <origin xyz="-0.032 0 0.070" rpy="0 0 0"/>
       <geometry>
-        <box size=".2 .2 .14"/>
+        <box size="0.20 0.20 0.143"/>
       </geometry>
     </collision>
@@ -48,5 +48,5 @@
       <origin xyz="0 0 0" rpy="0 0 0"/>
       <geometry>
-        <cylinder length=".026" radius=".0325"/>
+        <cylinder length="0.018" radius="0.033"/>
       </geometry>
     </collision>
@@ -76,5 +76,5 @@
       <origin xyz="0 0 0" rpy="0 0 0"/>
       <geometry>
-        <cylinder length=".026" radius=".0325"/>
+        <cylinder length="0.018" radius="0.033"/>
       </geometry>
     </collision>
@@ -140,28 +140,3 @@
     </inertial>
   </link>
-  <joint name="camera_joint" type="fixed">
-    <origin xyz="0.073 -0.011 0.084" rpy="0 0 0"/>
-    <parent link="base_link"/>
-    <child link="camera_link"/>
-  </joint>
-  <link name="camera_link">
-    <collision>
-      <origin xyz="0.005 0.011 0.013" rpy="0 0 0"/>
-      <geometry>
-        <box size="0.015 0.030 0.027"/>
-      </geometry>
-    </collision>
-  </link>
-  <joint name="camera_rgb_joint" type="fixed">
-    <origin xyz="0.003 0.011 0.009" rpy="0 0 0"/>
-    <parent link="camera_link"/>
-    <child link="camera_rgb_frame"/>
-  </joint>
-  <link name="camera_rgb_frame"/>
-  <joint name="camera_rgb_optical_joint" type="fixed">
-    <origin xyz="0 0 0" rpy="-1.57 0 -1.57"/>
-    <parent link="camera_rgb_frame"/>
-    <child link="camera_rgb_optical_frame"/>
-  </joint>
-  <link name="camera_rgb_optical_frame"/>
 </robot>

Commit message: add model collision

File: ros/src/robot/robot_description/urdf/robot_thesis.urdf.xacro (robot description, xacro)
@@ -11,5 +11,5 @@
   <link name="base_link">
     <visual>
-      <origin xyz="-0.032 0 0.0525" rpy="0 0 -1.5707"/>
+      <origin xyz="-0.0 0 0.0525" rpy="0 0 -1.5707"/>
       <geometry>
         <mesh filename="package://robot_description/meshes/stl/robot_base.stl" scale="0.001 0.001 0.001"/>
@@ -18,5 +18,5 @@
     </visual>
     <collision>
-      <origin xyz="-0.032 0 0.070" rpy="0 0 0"/>
+      <origin xyz="-0.0 0 0.070" rpy="0 0 0"/>
       <geometry>
         <box size="0.20 0.20 0.143"/>
@@ -116,5 +116,5 @@
     <parent link="base_link"/>
     <child link="base_scan"/>
-    <origin xyz="-0.032 0 0.172" rpy="0 0 0"/>
+    <origin xyz="0.0 0 0.172" rpy="0 0 0"/>
   </joint>
   <link name="base_scan">
@@ -127,7 +127,7 @@
     </visual> -->
     <collision>
-      <origin xyz="0.015 0 -0.0065" rpy="0 0 0"/>
+      <origin xyz="0.0 0 0.05" rpy="0 0 0"/>
       <geometry>
-        <cylinder length="0.0315" radius="0.055"/>
+        <cylinder length="0.0315" radius="0.035"/>
       </geometry>
     </collision>

Commit message: update body collision

File: ros/src/robot/robot_description/urdf/robot_thesis.urdf.xacro (robot description, xacro)
@@ -18,7 +18,7 @@
     </visual>
     <collision>
-      <origin xyz="-0.0 0 0.070" rpy="0 0 0"/>
+      <origin xyz="-0.0 0 0.11" rpy="0 0 0"/>
       <geometry>
-        <box size="0.20 0.20 0.143"/>
+        <cylinder length="0.11" radius="0.1"/>
       </geometry>
     </collision>

Commit message: change camera position

File: ros/src/robot/robot_description/urdf/robot_thesis.urdf.xacro (robot description, xacro)
@@ -141,5 +141,5 @@
   </link>
   <joint name="camera_left_joint" type="fixed">
-    <origin xyz="0.073 -0.02 0.084" rpy="0 0 0"/>
+    <origin xyz="0.1 -0.02 0.12" rpy="0 0 0"/>
     <parent link="base_link"/>
     <child link="camera_left_link"/>
@@ -154,5 +154,5 @@
   </link>
     <joint name="camera_right_joint" type="fixed">
-    <origin xyz="0.073 0.02 0.084" rpy="0 0 0"/>
+    <origin xyz="0.1 0.02 0.12" rpy="0 0 0"/>
     <parent link="base_link"/>
     <child link="camera_right_link"/>

Commit message: remove stereo visual

File: ros/src/robot/robot_description/urdf/robot_thesis.urdf.xacro (robot description, xacro)
@@ -3,6 +3,4 @@
   <xacro:include filename="$(find robot_description)/urdf/common_properties.xacro"/>
   <xacro:include filename="$(find robot_description)/urdf/robot_thesis.gazebo.xacro"/>
-  <xacro:include filename="$(find turtlebot_description)/urdf/turtlebot_gazebo.urdf.xacro"/>
-  <xacro:include filename="$(find turtlebot_description)/urdf/turtlebot_properties.urdf.xacro"/>
   <xacro:property name="r200_cam_rgb_px" value="0.005"/>
   <xacro:property name="r200_cam_rgb_py" value="0.018"/>
@@ -11,5 +9,10 @@
   <xacro:property name="parent" value="base_link"/>
   <xacro:property name="M_PI" value="3.14"/>
-    <xacro:property name="kinect_cam_py" value="-0.0125"/>
+  <xacro:property name="kinect_cam_py" value="-0.0125"/>
+  <xacro:property name="cam_px" value="-0.087" />
+  <xacro:property name="cam_pz" value="0.2870" />
+  <xacro:property name="cam_or" value="0" />
+  <xacro:property name="cam_op" value="0" />
+  <xacro:property name="cam_oy" value="0" />
   <link name="base_footprint"/>
   <joint name="base_joint" type="fixed">
@@ -193,10 +196,10 @@
     </joint>
       <link name="camera_link">
-      <visual>
+<!--       <visual>
        <origin xyz="0 0 0" rpy="0 0 ${M_PI/2}"/>
         <geometry>
          <mesh filename="package://turtlebot_description/meshes/sensors/kinect.dae"/>
         </geometry>
-      </visual>
+      </visual> -->
       <collision>
         <origin xyz="0.0 0.0 0.0" rpy="0 0 0"/>
