Commit message: add camera simulation

File: ros/src/robot/robot_description/urdf/robot_thesis.gazebo.xacro (robot description, xacro)
@@ -3,4 +3,5 @@
   <xacro:arg name="laser_visual" default="false"/>
   <xacro:arg name="imu_visual"   default="false"/>
+  <xacro:arg name="camera_visual" default="false"/>
   <gazebo reference="base_link">
     <material>Gazebo/DarkGrey</material>
@@ -124,3 +125,35 @@
     </sensor>
   </gazebo>
+   <gazebo reference="camera_rgb_frame">
+    <sensor type="camera" name="Pi Camera">
+      <always_on>true</always_on>
+      <visualize>$(arg camera_visual)</visualize>
+      <camera>
+          <horizontal_fov>1.085595</horizontal_fov>
+          <image>
+              <width>640</width>
+              <height>480</height>
+              <format>R8G8B8</format>
+          </image>
+          <clip>
+              <near>0.03</near>
+              <far>100</far>
+          </clip>
+      </camera>
+      <plugin name="camera_controller" filename="libgazebo_ros_camera.so">
+        <alwaysOn>true</alwaysOn>
+        <updateRate>30.0</updateRate>
+        <cameraName>src</cameraName>
+        <frameName>camera_rgb_optical_frame</frameName>
+        <imageTopicName>image</imageTopicName>
+        <cameraInfoTopicName>rgb/camera_info</cameraInfoTopicName>
+        <hackBaseline>0.07</hackBaseline>
+        <distortionK1>0.0</distortionK1>
+        <distortionK2>0.0</distortionK2>
+        <distortionK3>0.0</distortionK3>
+        <distortionT1>0.0</distortionT1>
+        <distortionT2>0.0</distortionT2>
+      </plugin>
+    </sensor>
+  </gazebo>
 </robot>

File: ros/src/robot/robot_description/urdf/robot_thesis.urdf.xacro (robot description, xacro)
@@ -140,3 +140,28 @@
     </inertial>
   </link>
+  <joint name="camera_joint" type="fixed">
+    <origin xyz="0.073 -0.011 0.084" rpy="0 0 0"/>
+    <parent link="base_link"/>
+    <child link="camera_link"/>
+  </joint>
+  <link name="camera_link">
+    <collision>
+      <origin xyz="0.005 0.011 0.013" rpy="0 0 0"/>
+      <geometry>
+        <box size="0.015 0.030 0.027"/>
+      </geometry>
+    </collision>
+  </link>
+  <joint name="camera_rgb_joint" type="fixed">
+    <origin xyz="0.003 0.011 0.009" rpy="0 0 0"/>
+    <parent link="camera_link"/>
+    <child link="camera_rgb_frame"/>
+  </joint>
+  <link name="camera_rgb_frame"/>
+  <joint name="camera_rgb_optical_joint" type="fixed">
+    <origin xyz="0 0 0" rpy="-1.57 0 -1.57"/>
+    <parent link="camera_rgb_frame"/>
+    <child link="camera_rgb_optical_frame"/>
+  </joint>
+  <link name="camera_rgb_optical_frame"/>
 </robot>

Commit message: add camerrgb & gray camera

File: ros/src/robot/robot_description/urdf/robot_thesis.gazebo.xacro (robot description, xacro)
@@ -125,5 +125,37 @@
     </sensor>
   </gazebo>
-   <gazebo reference="camera_rgb_frame">
+   <gazebo reference="camera_gray_link">
+    <sensor type="camera" name="Pi Camera">
+      <always_on>true</always_on>
+      <visualize>$(arg camera_visual)</visualize>
+      <camera>
+          <horizontal_fov>1.085595</horizontal_fov>
+          <image>
+              <width>640</width>
+              <height>480</height>
+              <format>L8</format>
+          </image>
+          <clip>
+              <near>0.03</near>
+              <far>100</far>
+          </clip>
+      </camera>
+      <plugin name="camera_controller" filename="libgazebo_ros_camera.so">
+        <alwaysOn>true</alwaysOn>
+        <updateRate>30.0</updateRate>
+        <cameraName>sensor/camera/grayscale/left</cameraName>
+        <frameName>camera_gray_link</frameName>
+        <imageTopicName>image_rect_g</imageTopicName>
+        <cameraInfoTopicName>camera_info</cameraInfoTopicName>
+        <hackBaseline>0.07</hackBaseline>
+        <distortionK1>0.0</distortionK1>
+        <distortionK2>0.0</distortionK2>
+        <distortionK3>0.0</distortionK3>
+        <distortionT1>0.0</distortionT1>
+        <distortionT2>0.0</distortionT2>
+      </plugin>
+    </sensor>
+  </gazebo>
+  <gazebo reference="camera_rgb_link">
     <sensor type="camera" name="Pi Camera">
       <always_on>true</always_on>
@@ -144,8 +176,8 @@
         <alwaysOn>true</alwaysOn>
         <updateRate>30.0</updateRate>
-        <cameraName>src</cameraName>
-        <frameName>camera_rgb_optical_frame</frameName>
-        <imageTopicName>image</imageTopicName>
-        <cameraInfoTopicName>rgb/camera_info</cameraInfoTopicName>
+        <cameraName>sensor/camera/color/left</cameraName>
+        <frameName>camera_rgb_link</frameName>
+        <imageTopicName>image_rect</imageTopicName>
+        <cameraInfoTopicName>camera_info</cameraInfoTopicName>
         <hackBaseline>0.07</hackBaseline>
         <distortionK1>0.0</distortionK1>

File: ros/src/robot/robot_description/urdf/robot_thesis.urdf.xacro (robot description, xacro)
@@ -140,12 +140,12 @@
     </inertial>
   </link>
-  <joint name="camera_joint" type="fixed">
-    <origin xyz="0.073 -0.011 0.084" rpy="0 0 0"/>
+  <joint name="camera_gray_joint" type="fixed">
+    <origin xyz="0.09 -0.04 0.13" rpy="0 0 0"/>
     <parent link="base_link"/>
-    <child link="camera_link"/>
+    <child link="camera_gray_link"/>
   </joint>
-  <link name="camera_link">
+  <link name="camera_gray_link">
     <collision>
-      <origin xyz="0.005 0.011 0.013" rpy="0 0 0"/>
+      <origin xyz="0 0 0" rpy="0 0 0"/>
       <geometry>
         <box size="0.015 0.030 0.027"/>
@@ -153,15 +153,16 @@
     </collision>
   </link>
-  <joint name="camera_rgb_joint" type="fixed">
-    <origin xyz="0.003 0.011 0.009" rpy="0 0 0"/>
-    <parent link="camera_link"/>
-    <child link="camera_rgb_frame"/>
+    <joint name="camera_rgb_joint" type="fixed">
+    <origin xyz="0.09 0.04 0.13" rpy="0 0 0"/>
+    <parent link="base_link"/>
+    <child link="camera_rgb_link"/>
   </joint>
-  <link name="camera_rgb_frame"/>
-  <joint name="camera_rgb_optical_joint" type="fixed">
-    <origin xyz="0 0 0" rpy="-1.57 0 -1.57"/>
-    <parent link="camera_rgb_frame"/>
-    <child link="camera_rgb_optical_frame"/>
-  </joint>
-  <link name="camera_rgb_optical_frame"/>
+  <link name="camera_rgb_link">
+    <collision>
+      <origin xyz="0 0 0" rpy="0 0 0"/>
+      <geometry>
+        <box size="0.015 0.030 0.027"/>
+      </geometry>
+    </collision>
+  </link>
 </robot>

Commit message: add camera

File: ros/src/robot/robot_description/urdf/robot_thesis.gazebo.xacro (robot description, xacro)
@@ -125,3 +125,35 @@
     </sensor>
   </gazebo>
+  <gazebo reference="camera_rgb_frame">
+    <sensor type="camera" name="Camera">
+      <always_on>true</always_on>
+      <visualize>$(arg camera_visual)</visualize>
+      <camera>
+          <horizontal_fov>1.085595</horizontal_fov>
+          <image>
+              <width>640</width>
+              <height>480</height>
+              <format>R8G8B8</format>
+          </image>
+          <clip>
+              <near>0.03</near>
+              <far>100</far>
+          </clip>
+      </camera>
+      <plugin name="camera_controller" filename="libgazebo_ros_camera.so">
+        <alwaysOn>true</alwaysOn>
+        <updateRate>30.0</updateRate>
+        <cameraName>src</cameraName>
+        <frameName>camera_rgb_optical_frame</frameName>
+        <imageTopicName>image</imageTopicName>
+        <cameraInfoTopicName>rgb/camera_info</cameraInfoTopicName>
+        <hackBaseline>0.07</hackBaseline>
+        <distortionK1>0.0</distortionK1>
+        <distortionK2>0.0</distortionK2>
+        <distortionK3>0.0</distortionK3>
+        <distortionT1>0.0</distortionT1>
+        <distortionT2>0.0</distortionT2>
+      </plugin>
+    </sensor>
+  </gazebo>
 </robot>

File: ros/src/robot/robot_description/urdf/robot_thesis.urdf.xacro (robot description, xacro)
@@ -140,3 +140,28 @@
     </inertial>
   </link>
+  <joint name="camera_joint" type="fixed">
+    <origin xyz="0.073 -0.011 0.084" rpy="0 0 0"/>
+    <parent link="base_link"/>
+    <child link="camera_link"/>
+  </joint>
+  <link name="camera_link">
+    <collision>
+      <origin xyz="0.005 0.011 0.013" rpy="0 0 0"/>
+      <geometry>
+        <box size="0.015 0.030 0.027"/>
+      </geometry>
+    </collision>
+  </link>
+  <joint name="camera_rgb_joint" type="fixed">
+    <origin xyz="0.003 0.011 0.009" rpy="0 0 0"/>
+    <parent link="camera_link"/>
+    <child link="camera_rgb_frame"/>
+  </joint>
+  <link name="camera_rgb_frame"/>
+  <joint name="camera_rgb_optical_joint" type="fixed">
+    <origin xyz="0 0 0" rpy="-1.57 0 -1.57"/>
+    <parent link="camera_rgb_frame"/>
+    <child link="camera_rgb_optical_frame"/>
+  </joint>
+  <link name="camera_rgb_optical_frame"/>
 </robot>

Commit message: add 2 mono camera

File: ros/src/robot/robot_description/urdf/robot_thesis.gazebo.xacro (robot description, xacro)
@@ -125,6 +125,6 @@
     </sensor>
   </gazebo>
-  <gazebo reference="camera_rgb_frame">
-    <sensor type="camera" name="Camera">
+  <gazebo reference="camera_left_link">
+    <sensor type="camera" name="camera_left">
       <always_on>true</always_on>
       <visualize>$(arg camera_visual)</visualize>
@@ -144,6 +144,38 @@
         <alwaysOn>true</alwaysOn>
         <updateRate>30.0</updateRate>
-        <cameraName>camera</cameraName>
-        <frameName>camera_rgb_optical_frame</frameName>
+        <cameraName>camera_left</cameraName>
+        <frameName>camera_left_link</frameName>
+        <imageTopicName>rgb/image_raw</imageTopicName>
+        <cameraInfoTopicName>rgb/camera_info</cameraInfoTopicName>
+        <hackBaseline>0.07</hackBaseline>
+        <distortionK1>0.0</distortionK1>
+        <distortionK2>0.0</distortionK2>
+        <distortionK3>0.0</distortionK3>
+        <distortionT1>0.0</distortionT1>
+        <distortionT2>0.0</distortionT2>
+      </plugin>
+    </sensor>
+  </gazebo>
+    <gazebo reference="camera_right_link">
+    <sensor type="camera" name="camera_right">
+      <always_on>true</always_on>
+      <visualize>$(arg camera_visual)</visualize>
+      <camera>
+          <horizontal_fov>1.085595</horizontal_fov>
+          <image>
+              <width>640</width>
+              <height>480</height>
+              <format>R8G8B8</format>
+          </image>
+          <clip>
+              <near>0.03</near>
+              <far>100</far>
+          </clip>
+      </camera>
+      <plugin name="camera_controller" filename="libgazebo_ros_camera.so">
+        <alwaysOn>true</alwaysOn>
+        <updateRate>30.0</updateRate>
+        <cameraName>camera_right</cameraName>
+        <frameName>camera_right_link</frameName>
         <imageTopicName>rgb/image_raw</imageTopicName>
         <cameraInfoTopicName>rgb/camera_info</cameraInfoTopicName>

File: ros/src/robot/robot_description/urdf/robot_thesis.urdf.xacro (robot description, xacro)
@@ -140,12 +140,12 @@
     </inertial>
   </link>
-  <joint name="camera_joint" type="fixed">
-    <origin xyz="0.073 -0.011 0.084" rpy="0 0 0"/>
+  <joint name="camera_left_joint" type="fixed">
+    <origin xyz="0.073 -0.02 0.084" rpy="0 0 0"/>
     <parent link="base_link"/>
-    <child link="camera_link"/>
+    <child link="camera_left_link"/>
   </joint>
-  <link name="camera_link">
+  <link name="camera_left_link">
     <collision>
-      <origin xyz="0.005 0.011 0.013" rpy="0 0 0"/>
+      <origin xyz="0.005 -0.02 0.013" rpy="0 0 0"/>
       <geometry>
         <box size="0.015 0.030 0.027"/>
@@ -153,15 +153,16 @@
     </collision>
   </link>
-  <joint name="camera_rgb_joint" type="fixed">
-    <origin xyz="0.003 0.011 0.009" rpy="0 0 0"/>
-    <parent link="camera_link"/>
-    <child link="camera_rgb_frame"/>
+    <joint name="camera_right_joint" type="fixed">
+    <origin xyz="0.073 0.02 0.084" rpy="0 0 0"/>
+    <parent link="base_link"/>
+    <child link="camera_right_link"/>
   </joint>
-  <link name="camera_rgb_frame"/>
-  <joint name="camera_rgb_optical_joint" type="fixed">
-    <origin xyz="0 0 0" rpy="-1.57 0 -1.57"/>
-    <parent link="camera_rgb_frame"/>
-    <child link="camera_rgb_optical_frame"/>
-  </joint>
-  <link name="camera_rgb_optical_frame"/>
+  <link name="camera_right_link">
+    <collision>
+      <origin xyz="0.005 0.02 0.013" rpy="0 0 0"/>
+      <geometry>
+        <box size="0.015 0.030 0.027"/>
+      </geometry>
+    </collision>
+  </link>
 </robot>

Commit message: add stereo camera

File: ros/src/robot/robot_description/urdf/robot_thesis.gazebo.xacro (robot description, xacro)
@@ -189,3 +189,39 @@
     </sensor>
   </gazebo>
+  <gazebo reference="camera_link">
+      <sensor type="depth" name="camera">
+        <always_on>true</always_on>
+        <update_rate>20.0</update_rate>
+        <camera>
+          <horizontal_fov>${60.0*3.14/180.0}</horizontal_fov>
+          <image>
+            <format>B8G8R8</format>
+            <width>640</width>
+            <height>480</height>
+          </image>
+          <clip>
+            <near>0.05</near>
+            <far>8.0</far>
+          </clip>
+        </camera>
+        <plugin name="kinect_camera_controller" filename="libgazebo_ros_openni_kinect.so">
+          <cameraName>camera</cameraName>
+          <alwaysOn>true</alwaysOn>
+          <updateRate>10</updateRate>
+          <imageTopicName>rgb/image_raw</imageTopicName>
+          <depthImageTopicName>depth/image_raw</depthImageTopicName>
+          <pointCloudTopicName>depth/points</pointCloudTopicName>
+          <cameraInfoTopicName>rgb/camera_info</cameraInfoTopicName>
+          <depthImageCameraInfoTopicName>depth/camera_info</depthImageCameraInfoTopicName>
+          <frameName>camera_depth_optical_frame</frameName>
+          <baseline>0.1</baseline>
+          <distortion_k1>0.0</distortion_k1>
+          <distortion_k2>0.0</distortion_k2>
+          <distortion_k3>0.0</distortion_k3>
+          <distortion_t1>0.0</distortion_t1>
+          <distortion_t2>0.0</distortion_t2>
+          <pointCloudCutoff>0.4</pointCloudCutoff>
+        </plugin>
+      </sensor>
+    </gazebo>
 </robot>

File: ros/src/robot/robot_description/urdf/robot_thesis.urdf.xacro (robot description, xacro)
@@ -3,4 +3,13 @@
   <xacro:include filename="$(find robot_description)/urdf/common_properties.xacro"/>
   <xacro:include filename="$(find robot_description)/urdf/robot_thesis.gazebo.xacro"/>
+  <xacro:include filename="$(find turtlebot_description)/urdf/turtlebot_gazebo.urdf.xacro"/>
+  <xacro:include filename="$(find turtlebot_description)/urdf/turtlebot_properties.urdf.xacro"/>
+  <xacro:property name="r200_cam_rgb_px" value="0.005"/>
+  <xacro:property name="r200_cam_rgb_py" value="0.018"/>
+  <xacro:property name="r200_cam_rgb_pz" value="0.013"/>
+  <xacro:property name="r200_cam_depth_offset" value="0.01"/>
+  <xacro:property name="parent" value="base_link"/>
+  <xacro:property name="M_PI" value="3.14"/>
+    <xacro:property name="kinect_cam_py" value="-0.0125"/>
   <link name="base_footprint"/>
   <joint name="base_joint" type="fixed">
@@ -166,3 +175,49 @@
     </collision>
   </link>
+    <joint name="camera_rgb_joint" type="fixed">
+      <origin xyz="${cam_px} ${kinect_cam_py} ${cam_pz}" rpy="${cam_or} ${cam_op} ${cam_oy}"/>
+      <parent link="${parent}"/>
+      <child link="camera_rgb_frame" />
+    </joint>
+    <link name="camera_rgb_frame"/>
+    <joint name="camera_rgb_optical_joint" type="fixed">
+      <origin xyz="0 0 0" rpy="${-M_PI/2} 0 ${-M_PI/2}" />
+      <parent link="camera_rgb_frame" />
+      <child link="camera_rgb_optical_frame" />
+    </joint>
+    <link name="camera_rgb_optical_frame"/>
+    <joint name="camera_joint" type="fixed">
+      <origin xyz="-0.031 ${-kinect_cam_py} -0.016" rpy="0 0 0"/>
+      <parent link="camera_rgb_frame"/>
+      <child link="camera_link"/>
+    </joint>
+      <link name="camera_link">
+      <visual>
+       <origin xyz="0 0 0" rpy="0 0 ${M_PI/2}"/>
+        <geometry>
+         <mesh filename="package://turtlebot_description/meshes/sensors/kinect.dae"/>
+        </geometry>
+      </visual>
+      <collision>
+        <origin xyz="0.0 0.0 0.0" rpy="0 0 0"/>
+        <geometry>
+          <box size="0.07271 0.27794 0.073"/>
+        </geometry>
+      </collision>
+    </link>
+    <!-- The fixed joints & links below are usually published by static_transformers launched by the OpenNi launch
+         files. However, for Gazebo simulation we need them, so we add them here.
+         (Hence, don't publish them additionally!) -->
+  <joint name="camera_depth_joint" type="fixed">
+    <origin xyz="0 ${2 * -kinect_cam_py} 0" rpy="0 0 0" />
+    <parent link="camera_rgb_frame" />
+    <child link="camera_depth_frame" />
+  </joint>
+  <link name="camera_depth_frame"/>
+  <joint name="camera_depth_optical_joint" type="fixed">
+    <origin xyz="0 0 0" rpy="${-M_PI/2} 0 ${-M_PI/2}" />
+    <parent link="camera_depth_frame" />
+    <child link="camera_depth_optical_frame" />
+  </joint>
+  <link name="camera_depth_optical_frame"/>
 </robot>

Commit message: add camera optical frames

File: ros/src/robot/robot_description/urdf/robot_thesis.gazebo.xacro (robot description, xacro)
@@ -125,5 +125,5 @@
     </sensor>
   </gazebo>
-  <gazebo reference="camera_left_link">
+  <gazebo reference="camera_left_rgb_frame">
     <sensor type="camera" name="camera_left">
       <always_on>true</always_on>
@@ -145,5 +145,5 @@
         <updateRate>30.0</updateRate>
         <cameraName>camera_left</cameraName>
-        <frameName>camera_left_link</frameName>
+        <frameName>camera_left_rgb_optical_frame</frameName>
         <imageTopicName>image_raw</imageTopicName>
         <cameraInfoTopicName>camera_info</cameraInfoTopicName>
@@ -157,5 +157,5 @@
     </sensor>
   </gazebo>
-    <gazebo reference="camera_right_link">
+    <gazebo reference="camera_right_rgb_frame">
     <sensor type="camera" name="camera_right">
       <always_on>true</always_on>
@@ -177,5 +177,5 @@
         <updateRate>30.0</updateRate>
         <cameraName>camera_right</cameraName>
-        <frameName>camera_right_link</frameName>
+        <frameName>camera_right_rgb_optical_frame</frameName>
         <imageTopicName>image_raw</imageTopicName>
         <cameraInfoTopicName>camera_info</cameraInfoTopicName>

File: ros/src/robot/robot_description/urdf/robot_thesis.urdf.xacro (robot description, xacro)
@@ -165,4 +165,16 @@
     </collision>
   </link>
+  <joint name="camera_left_rgb_joint" type="fixed">
+    <origin xyz="0.003 0.02 0.009" rpy="0 0 0"/>
+    <parent link="camera_left_link"/>
+    <child link="camera_left_rgb_frame"/>
+  </joint>
+  <link name="camera_left_rgb_frame"/>
+  <joint name="camera_left_rgb_optical_joint" type="fixed">
+    <origin xyz="0 0 0" rpy="-1.57 0 -1.57"/>
+    <parent link="camera_left_rgb_frame"/>
+    <child link="camera_left_rgb_optical_frame"/>
+  </joint>
+  <link name="camera_left_rgb_optical_frame"/>
     <joint name="camera_right_joint" type="fixed">
     <origin xyz="0.1 0.02 0.12" rpy="0 0 0"/>
@@ -178,4 +190,16 @@
     </collision>
   </link>
+    <joint name="camera_right_rgb_joint" type="fixed">
+    <origin xyz="0.003 0.02 0.009" rpy="0 0 0"/>
+    <parent link="camera_right_link"/>
+    <child link="camera_right_rgb_frame"/>
+  </joint>
+  <link name="camera_right_rgb_frame"/>
+  <joint name="camera_right_rgb_optical_joint" type="fixed">
+    <origin xyz="0 0 0" rpy="-1.57 0 -1.57"/>
+    <parent link="camera_right_rgb_frame"/>
+    <child link="camera_right_rgb_optical_frame"/>
+  </joint>
+  <link name="camera_right_rgb_optical_frame"/>
     <joint name="camera_rgb_joint" type="fixed">
       <origin xyz="${cam_px} ${kinect_cam_py} ${cam_pz}" rpy="${cam_or} ${cam_op} ${cam_oy}"/>
